File: power.kicad_sch (KiCad schematic)
At the start: 13 parts, among them U2 AP2112K-3.3

Commit message: Power rail stuff
Parts:
- removed C4, C5: 1u, symbol Device:C_Small
- removed U2: AP2112K-3.3, Package_TO_SOT_SMD:SOT-23-5, symbol Regulator_Linear:AP2112K-3.3
- added C13: 4.7u, symbol Device:C_Small
- added C14: 10u, symbol Device:C_Small
- added C15: 6.8p, symbol Device:C_Small
- added L4: 2.2u, symbol Device:L
- added R7: 150k, symbol Device:R_US
- added R8: 33.2k, symbol Device:R_US
- added U4: TLV62569DBV, Package_TO_SOT_SMD:SOT-23-5, symbol Regulator_Switching:TLV62569DBV
Connections:
- net +3.3V: now also C14.1, C15.2, L4.2, R7.1
- net +5V: now also C13.1, U4.1 (EN), U4.4 (VIN)
- net GND: now also C13.2, C14.2, R8.2, U4.2 (GND)
- new net: C15.1, R7.2, R8.1, U4.5 (FB)
- new net: L4.1, U4.3 (SW)
Other:
- moved on the sheet: TP2, TP3

Commit message: Fixed regulator, started wiring the microSD & MCU
Parts:
- added C4: 4.7u, symbol Device:C_Small
- added R9: 150k, symbol Device:R_US
- R7: value 150k -> 300k
- R8: value 33.2k -> 100k
Connections:
- net +3.3V: now also R9.1; no longer R7.1
- net GND: now also C4.2
- net VBUS: now also C4.1
- new net: R7.1, R9.2
Other:
- note added: "1.5Mhz"
- note added: "ferrite value calc"
- moved on the sheet: C14, C3, C6, D2, D3, L1, R2, R3, TP2, TP3

Commit message: MCU wiring
Connections:
- net BUCK_FB: now reaches C15.1, R7.2, R8.1, U4.5 (FB)
- net BUCK_SW: now reaches L4.1, U4.3 (SW)
Other:
- moved on the sheet: C14, C15, L4, R7, R8, R9

Commit message: Minor re-organization and additional power filtering
Parts:
- added C37: 4.7u, symbol Device:C_Small
- added C38: 10u, symbol Device:C_Small
Connections:
- net +3.3V: now also C37.1, C38.1
- net GND: now also C37.2, C38.2

Commit message: Minor
Parts:
- added D5: GREEN, LED_SMD:LED_0805_2012Metric, symbol Device:LED
- added R12: 560, symbol Device:R_US
- added R13: 100k, symbol Device:R_US
- added SW1: SW_SPDT, symbol Switch:SW_SPDT
Connections:
- net +5V: now also SW1.3 (C); no longer U4.1 (EN)
- net GND: now also D5.1 (K), R13.2
- net VBUS: now also R12.1
- new net: R13.1, SW1.2 (B), U4.1 (EN)
- new net: D5.2 (A), R12.2
Other:
- moved on the sheet: C13, C14, C15, C37, C38, D2, D3, L4, R2, R3, R7, R8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

Commit message: A lot re-wiring, added appropriate parts for schematic components. Some re-organization.
Parts:
- removed C15: 6.8p, symbol Device:C_Small
- C14: value 10u -> 10n
- U4: value TLV62569DBV -> TLV62569DBVR
Connections:
- net BUCK_FB is gone; now on net +3.3V: R7.2, R8.1, U4.5 (FB)
Other:
- moved on the sheet: C37, C38

Commit message: Alot of stuff
Parts:
- removed SW1: SW_SPDT, symbol Switch:SW_SPDT
- added SW1: SLW-116641-3A-RA-S-D, SamacSys_Parts:SLW1166413ARASD, symbol advres:SW_SPDT
- D2: value GREEN -> 5V_GOOD
- D3: value GREEN -> 3V3_GOOD
- D5: value GREEN -> VBUS_GOOD
Connections:
- net +5V: now also SW1.3 (C)
- net at R13.1, U4.1 (EN): now also SW1.2 (B)
Other:
- moved on the sheet: D2, D3, R2, R3, TP2, TP3

Commit message: Stuff
Parts:
- removed D2: 5V_GOOD, LED_SMD:LED_0805_2012Metric, symbol Device:LED
- removed D3: 3V3_GOOD, LED_SMD:LED_0805_2012Metric, symbol Device:LED
- removed D5: VBUS_GOOD, LED_SMD:LED_0805_2012Metric, symbol Device:LED
- added D10: VBUS_GOOD, SamacSys_Parts:LEDC2012X110N, symbol Device:LED
- added D11: 5V_GOOD, SamacSys_Parts:LEDC2012X110N, symbol Device:LED
- added D12: 3V3_GOOD, SamacSys_Parts:LEDC2012X110N, symbol Device:LED
- R12, R2: value 560 -> 180
- R3: value 220 -> 62
Connections:
- net GND: now also D10.1 (K), D11.1 (K), D12.1 (K)
- net at R2.2: now also D11.2 (A)
- net at R12.2: now also D10.2 (A)
- net at R3.2: now also D12.2 (A)
